File: _restore_backup_2026-09-23T11-23-55-188/esp_main_board.kicad_sch (KiCad schematic)
At the start: 70 parts, among them J1 USB_C_Receptacle_USB2.0_16P, J10 Screw_Terminal_01x02, J11 Conn_01x06_Socket, J12 Conn_01x03_Pin, J13 Raspberry_Pi_4, J14 Conn_01x04_Socket, J15 Screw_Terminal_01x02, J16 Screw_Terminal_01x02, J19 Conn_01x05_Socket, J2 Conn_01x03_Pin, J22 Conn_01x05_Socket, J3 Conn_01x03_Pin, J4 Conn_01x03_Pin, J5 Conn_01x03_Pin, J6 Conn_01x03_Socket, J7 Conn_01x03_Socket, J8 Conn_01x03_Socket, J9 Conn_01x03_Socket, Q3 BSS138, Q4 BSS138, Q5 BSS138, Q6 BSS138, Q7 BSS138, Q8 BSS138, SW1 SW_Push, SW2 SW_Push, U1 USBLC6-2SC6, U2 AMS1117-3.3, U3 ESP32-WROOM-32, U4 LM2596S-5, U5 CH340G, U6 TB6612FNG, U7 CD74HC4067M, Y1 Crystal_GND24

Commit message: feat: 3d pcb layout version 1 without imu
Parts:
- removed J16: Screw_Terminal_01x02, TerminalBlock_Phoenix:TerminalBlock_Phoenix_MPT-0,5-2-2.54_1x02_P2.54mm_Horizontal, symbol Connector:Screw_Terminal_01x02
- removed J19, J22: Conn_01x05_Socket, Connector_PinSocket_2.54mm:PinSocket_1x05_P2.54mm_Vertical, symbol Connector:Conn_01x05_Socket
- removed U4: LM2596S-5, Package_TO_SOT_SMD:TO-263-5_TabPin3, symbol Regulator_Switching:LM2596S-5
- removed U7: CD74HC4067M, Package_SO:SOIC-24W_7.5x15.4mm_P1.27mm, symbol 74xx:CD74HC4067M
Connections:
- net +5V: no longer J13.2 (5V), J13.4 (5V)
- net DC_A+: now also J15.2 (Pin_2); no longer J15.1 (Pin_1)
- net DC_A-: now also J15.1 (Pin_1); no longer J15.2 (Pin_2)
- net GND: no longer J13.14 (GND), J13.20 (GND), J13.25 (GND), J13.30 (GND), J13.34 (GND), J13.39 (GND), J13.6 (GND), J13.9 (GND)
- net +3.3V: no longer names the net of J13.1 (3V3), J13.17 (3V3)
- new net: J13.14 (GND), J13.20 (GND), J13.25 (GND), J13.30 (GND), J13.34 (GND), J13.39 (GND), J13.6 (GND), J13.9 (GND)
- new net: J13.2 (5V), J13.4 (5V)
- no-connect marks 45 -> 17
Other:
- note added: "Notes: 1 -"
- note added: "Notes: 1 - I have used AMS1117-3.3 voltage redulator. The circiut is copied as in the datasheet. 2 - Maybe use 4u7 capacitors as well to decrease the Bill of Materials."
- note added: "Notes: 1 - I have used PESD5V0L1ULD for esd. But in our stock we have BAT54C. I have search for it but i did not understand. How may we implement that component?"
- note added: "Notes: 1 - Ihave connected the 3.3V to the ESP with capacitors to stabize the 3.3V. They are decoupling capacitors. 2 - All the pins are labeled via global labels. 3 - Two buttons are added. One above is enable button. Some applications shows that we can connect enable button to directly GND via capacitors. 4- Second button is BOOT button. In order for the Chip Boot Mode, strapping pins GPIO0 and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"
- note removed: "12 - 5 - 3.3 - GND"
- moved on the sheet: C10, C11, C12, C13, C14, C15, C3, C4, J10, J11, J12, J13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
