File: _restore_backup_2026-09-23T11-23-55-188/little_daisies_dev_board.kicad_pcb (KiCad board)
At the start: 2 copper layers, 56 x 65 mm, 70 parts, among them J1 USB_C_Receptacle_USB2.0_16P, J10 Screw_Terminal_01x02, J11 Conn_01x06_Socket, J12 Conn_01x03_Pin, J13 Raspberry_Pi_4, J14 Conn_01x04_Socket, J15 Screw_Terminal_01x02, J16 Screw_Terminal_01x02, J19 Conn_01x05_Socket, J2 Conn_01x03_Pin, J22 Conn_01x05_Socket, J3 Conn_01x03_Pin, J4 Conn_01x03_Pin, J5 Conn_01x03_Pin, J6 Conn_01x03_Socket, J7 Conn_01x03_Socket, J8 Conn_01x03_Socket, J9 Conn_01x03_Socket, Q3 BSS138, Q4 BSS138, Q5 BSS138, Q6 BSS138, Q7 BSS138, Q8 BSS138, SW1 SW_Push, SW2 SW_Push, U1 USBLC6-2SC6, U2 AMS1117-3.3, U3 ESP32-WROOM-32, U4 LM2596S-5, U5 CH340G, U6 TB6612FNG, U7 CD74HC4067M, Y1 Crystal_GND24

Commit message: feat: 3d pcb layout version 1 without imu
Parts:
- removed J16: Screw_Terminal_01x02, TerminalBlock_Phoenix:TerminalBlock_Phoenix_MPT-0,5-2-2.54_1x02_P2.54mm_Horizontal
- removed J19, J22: Conn_01x05_Socket, Connector_PinSocket_2.54mm:PinSocket_1x05_P2.54mm_Vertical
- removed U4: LM2596S-5, Package_TO_SOT_SMD:TO-263-5_TabPin3
- removed U7: CD74HC4067M, Package_SO:SOIC-24W_7.5x15.4mm_P1.27mm
- moved C14 20.0 mm to (207.2, 106.9)
- moved C13 19.6 mm to (212.2, 107.2)
- moved Y1 19.6 mm to (209.6, 107.1)
- moved U5 19.4 mm to (212.4, 112.6)
- moved J10 18.5 mm to (190.4, 114.2)
- moved J15 17.9 mm to (190.4, 107.6)
- moved J2 17.9 mm to (188.6, 103.8)
- moved J4 16.8 mm to (188.6, 100.2)
- moved C10 16.4 mm to (206.4, 105.1)
- moved J3 16.1 mm to (188.6, 89.3)
- moved C12 15.8 mm to (205.8, 102.0), turned to 0 degrees
- moved J7 15.8 mm to (188.6, 96.5)
- moved J6 14.8 mm to (188.6, 93.0)
- moved U6 14.4 mm to (200.2, 105.7)
- moved R11 13.9 mm to (205.4, 105.1)
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Connections:
- net +3.3V renamed Net-(J13-3V3-Pad1)
- J13 pad 14: GND -> Net-(J13-GND-Pad14)
- J13 pad 2: +5V -> Net-(J13-5V-Pad2)
- J13 pad 20: GND -> Net-(J13-GND-Pad14)
- J13 pad 25: GND -> Net-(J13-GND-Pad14)
- J13 pad 30: GND -> Net-(J13-GND-Pad14)
- J13 pad 34: GND -> Net-(J13-GND-Pad14)
- J13 pad 39: GND -> Net-(J13-GND-Pad14)
- J13 pad 4: +5V -> Net-(J13-5V-Pad2)
- J13 pad 6: GND -> Net-(J13-GND-Pad14)
- J13 pad 9: GND -> Net-(J13-GND-Pad14)
- J15 pad 1: /ESP_main_board/DC_A+ -> /ESP_main_board/DC_A-
- J15 pad 2: /ESP_main_board/DC_A- -> /ESP_main_board/DC_A+
Other:
- board text removed: "+3V3"
- board text removed: "+5V"
- board text removed: "3V3<--->5V"
- board text removed: "GND"
