File: _restore_backup_2026-10-09T12-16-25-202/esp_main_board.kicad_sch (KiCad schematic)
At the start: 70 parts, among them J1 USB_C_Receptacle_USB2.0_16P, J10 Screw_Terminal_01x02, J11 Conn_01x06_Socket, J12 Conn_01x03_Pin, J13 Raspberry_Pi_4, J14 Conn_01x04_Socket, J15 Screw_Terminal_01x02, J16 Screw_Terminal_01x02, J19 Conn_01x05_Socket, J2 Conn_01x03_Pin, J22 Conn_01x05_Socket, J3 Conn_01x03_Pin, J4 Conn_01x03_Pin, J5 Conn_01x03_Pin, J6 Conn_01x03_Socket, J7 Conn_01x03_Socket, J8 Conn_01x03_Socket, J9 Conn_01x03_Socket, Q3 BSS138, Q4 BSS138, Q5 BSS138, Q6 BSS138, Q7 BSS138, Q8 BSS138, SW1 SW_Push, SW2 SW_Push, U1 USBLC6-2SC6, U2 AMS1117-3.3, U3 ESP32-WROOM-32, U4 LM2596S-5, U5 CH340G, U6 TB6612FNG, U7 CD74HC4067M, Y1 Crystal_GND24

Commit message: feat: 3d pcb layout version 1 without imu
Parts:
- removed U7: CD74HC4067M, Package_SO:SOIC-24W_7.5x15.4mm_P1.27mm, symbol 74xx:CD74HC4067M
Changed lines of the file:
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@@
-	)
-	(symbol
-		(lib_id "74xx:CD74HC4067M")
-		(at 173.99 248.92 0)
-		(unit 1)
-		(body_style 1)
-		(exclude_from_sim no)
-		(in_bom yes)
-		(on_board yes)
-		(in_pos_files yes)
-		(dnp no)
-		(fields_autoplaced yes)
-		(property "Reference" "U7"
-			(at 176.1333 222.25 0)
-			(show_name no)
-			(do_not_autoplace no)
-			(effects
-				(font
-					(size 1.27 1.27)
-				)
-				(justify left)
-			)
-		)
-		(property "Value" "CD74HC4067M"
-			(at 176.1333 224.79 0)
-			(show_name no)
-			(do_not_autoplace no)
-			(effects
-				(font
-					(size 1.27 1.27)
-				)
-				(justify left)
-			)
-		)
-		(property "Footprint" "Package_SO:SOIC-24W_7.5x15.4mm_P1.27mm"
-			(at 196.85 274.32 0)
-			(hide yes)
-			(show_name no)
-			(do_not_autoplace no)
-			(effects
-				(font
-					(size 1.27 1.27)
-					(italic yes)
-				)
-			)
-		)
-		(property "Datasheet" "http://www.ti.com/lit/ds/symlink/cd74hc4067.pdf"
-			(at 165.1 227.33 0)
-			(hide yes)
-			(show_name no)
-			(do_not_autoplace no)
-			(effects
-				(font
-					(size 1.27 1.27)
-				)
-			)
-		)
-		(property "Description" "High-Speed CMOS Logic 16-Channel Analog Multiplexer/Demultiplexer, SOIC-24"
-			(at 173.99 248.92 0)
-			(hide yes)
-			(show_name no)
-			(do_not_autoplace no)
-			(effects
-				(font
-					(size 1.27 1.27)
-				)
-			)
-		)
-		(pin "3"
-		)
-		(pin "13"
-		)
-		(pin "21"
-		)
-		(pin "9"
-		)
-		(pin "24"
-		)
-		(pin "5"
-		)
-		(pin "23"
-		)
-		(pin "8"
-		)
-		(pin "15"
-		)
-		(pin "14"
-		)
-		(pin "1"
-		)
-		(pin "20"
-		)
-		(pin "22"
-		)
-		(pin "19"
-		)
-		(pin "17"
-		)
-		(pin "18"
-		)
-		(pin "2"
-		)
-		(pin "4"
-		)
-		(pin "10"
-		)
-		(pin "11"
-		)
-		(pin "12"
-		)
-		(pin "16"
-		)
-		(pin "6"
-		)
-		(pin "7"
-		)
-		(instances
-			(project "little_daisies_dev_board"
-				(path "/1d7f8a23-917d-4aaf-9484-e227942640a5/cfc3d48e-7a3b-4f9d-b699-4f7359090067"
-					(reference "U7")
-					(unit 1)
-				)
-			)
-		)
 	)
 	(symbol
