File: _restore_backup_2026-10-09T12-16-25-202/little_daisies_dev_board.kicad_pcb (KiCad board)
At the start: 2 copper layers, 56 x 65 mm, 70 parts, among them J1 USB_C_Receptacle_USB2.0_16P, J10 Screw_Terminal_01x02, J11 Conn_01x06_Socket, J12 Conn_01x03_Pin, J13 Raspberry_Pi_4, J14 Conn_01x04_Socket, J15 Screw_Terminal_01x02, J16 Screw_Terminal_01x02, J19 Conn_01x05_Socket, J2 Conn_01x03_Pin, J22 Conn_01x05_Socket, J3 Conn_01x03_Pin, J4 Conn_01x03_Pin, J5 Conn_01x03_Pin, J6 Conn_01x03_Socket, J7 Conn_01x03_Socket, J8 Conn_01x03_Socket, J9 Conn_01x03_Socket, Q3 BSS138, Q4 BSS138, Q5 BSS138, Q6 BSS138, Q7 BSS138, Q8 BSS138, SW1 SW_Push, SW2 SW_Push, U1 USBLC6-2SC6, U2 AMS1117-3.3, U3 ESP32-WROOM-32, U4 LM2596S-5, U5 CH340G, U6 TB6612FNG, U7 CD74HC4067M, Y1 Crystal_GND24

Commit message: feat: 3d pcb layout version 1 without imu
Parts:
- removed U4: LM2596S-5, Package_TO_SOT_SMD:TO-263-5_TabPin3
- removed U7: CD74HC4067M, Package_SO:SOIC-24W_7.5x15.4mm_P1.27mm
